File: gsm_module/hardware/hardware.kicad_pcb (KiCad board)
At the start: 2 copper layers, 60 parts, among them J1 Screw_Terminal_01x04, J10 Conn_01x02_Male, J11 Conn_01x02_Male, J12 Conn_01x02_Male, J13 Conn_01x02_Male, J2 SIM800C Module, J3 SIM800C Module Side A, J4 Programming interface, J5 SWD Debugging Interface, J6 Conn_01x02_Male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

Commit message: rev 1.6 (changed SMT antenna)
Parts:
- removed J3: SIM800C Module Side A, Connector_PinHeader_1.27mm:PinHeader_1x06_P1.27mm_Vertical
- added AE1: MOLEX 734120114, its_app:KH-IPEX4-2020, F.Cu at (75.0, 19.5)
- added AE2: MOLEX 734120114, its_app:KH-IPEX4-2020, F.Cu at (71.7, 45.9)
- added C14: 7.5nF, Capacitor_THT:C_Disc_D4.3mm_W1.9mm_P5.00mm, F.Cu at (81.0, 57.0)
- added C15: 33pF, Capacitor_THT:C_Disc_D4.3mm_W1.9mm_P5.00mm, F.Cu at (84.0, 49.5)
- added R17: 10k, Resistor_THT:R_Axial_DIN0309_L9.0mm_D3.2mm_P12.70mm_Horizontal, F.Cu at (63.0, 60.0)
- added U6: SIM868, its_app:XCVR_SIM868, F.Cu at (79.5, 33.0)
- C11, C5: value 5nF -> 7.5nF
- J1: footprint Connector_PinHeader_1.27mm:PinHeader_1x04_P1.27mm_Vertical -> its_app:5mm Pitch Screw Terminal 1x04
- J2: value SIM800C Module -> 78646-3001; footprint Connector_PinHeader_1.27mm:PinHeader_1x06_P1.27mm_Vertical -> its_app:MOLEX_78646-3001
- moved D2 183.8 mm to (256.5, 172.5)
- moved C2 153.2 mm to (253.5, 150.0)
- moved L2 144.5 mm to (246.0, 159.0)
- moved U3 135.4 mm to (21.0, 120.0)
- moved R4 134.7 mm to (234.0, 148.5)
- moved R2 129.4 mm to (232.5, 172.5)
- moved U10 128.3 mm to (269.1, 156.8)
- moved C13 126.5 mm to (31.5, 111.0)
- moved C11 126.4 mm to (31.5, 103.5)
- moved U5 123.0 mm to (36.0, 121.5)
- moved C12 122.7 mm to (18.0, 139.5)
- moved C4 121.6 mm to (237.0, 157.5), turned to 270 degrees
- moved J6 119.0 mm to (88.5, 187.5)
- moved J8 117.4 mm to (31.5, 169.5)
- moved R13 116.2 mm to (192.0, 34.5)
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Connections:
- R9 pad 1: Net-(J2-Pad4) -> Net-(R9-Pad1)
- U4 pad 9: RESET_PIN -> SIM8xx_PWR_PIN
Other:
- net class 2A_PWR added: clearance 0.5, trace_width 0.75, via_dia 0.8, via_drill 0.4
